File: hardware/air_station_1v5/air_station_1v5.kicad_sch (KiCad schematic)
At the start: 40 parts, among them J1 SIM7200-6-0-18-00-X_REVA, J2 Micro_SD_Card, J4 BAT_PORT, J5 PROG_PORT, U1 A9G, U1 AP7312-1833, U2 MIC5225-3.3, U3 MCP73831-2-OT, U5 BMP388, X1 ENS160

Commit message: update 1.9
I2C pullups update
Parts:
- added R11, R12: 4.7K, Adafruit BMP388:0603-NO, symbol Adafruit BMP388-eagle-import:RESISTOR_0603_NOOUT
Connections:
- net 3.3V: now also R11.2, R12.2
- net I2C2_SCL: now also R12.1
- net I2C2_SDA: now also R11.1
Other:
- note added: "1.8 [e]"
- note removed: "1.1 [e]"
Changed lines of the file:
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@@
   (junction (at 86.36 248.92) (diameter 0) (color 0 0 0 0)
   )
+  (junction (at 48.26 49.53) (diameter 0) (color 0 0 0 0)
+  )
   (junction (at 210.82 186.69) (diameter 0) (color 0 0 0 0)
   )
@@
   (junction (at 311.15 143.51) (diameter 0) (color 0 0 0 0)
   )
+  (junction (at 44.45 52.07) (diameter 0) (color 0 0 0 0)
+  )
   (junction (at 182.88 265.43) (diameter 0) (color 0 0 0 0)
   )
@@
   (junction (at 43.18 97.79) (diameter 0) (color 0 0 0 0)
   )
+  (junction (at 25.4 49.53) (diameter 0) (color 0 0 0 0)
+  )
   (wire (pts (xy 86.36 57.15) (xy 90.17 57.15))
     (stroke (width 0.1524) (type solid))
@@
     (stroke (width 0) (type default))
   )
+  (wire (pts (xy 40.64 49.53) (xy 48.26 49.53))
+    (stroke (width 0) (type default))
+  )
   (wire (pts (xy 74.93 26.67) (xy 74.93 31.75))
     (stroke (width 0) (type default))
@@
     (stroke (width 0) (type default))
   )
+  (wire (pts (xy 30.48 52.07) (xy 25.4 52.07))
+    (stroke (width 0) (type default))
+  )
   (wire (pts (xy 72.39 31.75) (xy 72.39 26.67))
     (stroke (width 0.1524) (type solid))
@@
     (stroke (width 0) (type default))
   )
+  (wire (pts (xy 40.64 52.07) (xy 44.45 52.07))
+    (stroke (width 0) (type default))
+  )
   (wire (pts (xy 173.99 151.13) (xy 177.8 151.13))
     (stroke (width 0) (type default))
@@
     (stroke (width 0) (type default))
   )
+  (wire (pts (xy 44.45 52.07) (xy 53.34 52.07))
+    (stroke (width 0) (type default))
+  )
   (wire (pts (xy 43.18 106.68) (xy 43.18 107.95))
     (stroke (width 0.1524) (type solid))
@@
     (stroke (width 0) (type default))
   )
+  (wire (pts (xy 25.4 49.53) (xy 25.4 46.99))
+    (stroke (width 0) (type default))
+  )
   (wire (pts (xy 311.15 143.51) (xy 311.15 146.05))
     (stroke (width 0.1524) (type solid))
@@
     (stroke (width 0) (type default))
   )
+  (wire (pts (xy 30.48 49.53) (xy 25.4 49.53))
+    (stroke (width 0) (type default))
+  )
   (wire (pts (xy 372.11 77.47) (xy 336.55 77.47))
     (stroke (width 0.1524) (type solid))
@@
     (stroke (width 0) (type default))
   )
+  (wire (pts (xy 48.26 49.53) (xy 53.34 49.53))
+    (stroke (width 0) (type default))
+  )
   (wire (pts (xy 86.36 248.92) (xy 86.36 252.73))
     (stroke (width 0) (type default))
@@
     (stroke (width 0) (type default))
   )
+  (wire (pts (xy 25.4 52.07) (xy 25.4 49.53))
+    (stroke (width 0) (type default))
+  )
   (wire (pts (xy 86.36 255.27) (xy 88.9 255.27))
     (stroke (width 0) (type default))
   )
-  (wire (pts (xy 43.18 49.53) (xy 53.34 49.53))
-    (stroke (width 0) (type default))
-  )
   (wire (pts (xy 278.13 74.93) (xy 273.05 74.93))
     (stroke (width 0.1524) (type solid))
@@
     (stroke (width 0) (type default))
   )
+  (wire (pts (xy 44.45 43.18) (xy 44.45 52.07))
+    (stroke (width 0) (type default))
+  )
   (wire (pts (xy 120.65 49.53) (xy 128.27 49.53))
     (stroke (width 0) (type default))
@@
     (stroke (width 0.1524) (type solid))
   )
-  (wire (pts (xy 43.18 52.07) (xy 53.34 52.07))
-    (stroke (width 0) (type default))
-  )
   (wire (pts (xy 97.79 26.67) (xy 97.79 31.75))
     (stroke (width 0) (type default))
@@
   )
   (wire (pts (xy 147.32 200.66) (xy 156.21 200.66))
+    (stroke (width 0) (type default))
+  )
+  (wire (pts (xy 48.26 40.64) (xy 48.26 49.53))
     (stroke (width 0) (type default))
   )
@@
     (effects (font (size 2.1844 1.8567)) (justify left bottom))
   )
-  (text "1.1 [e]" (at 389.8241 280.9738 0)
+  (text "1.8 [e]" (at 391.16 280.67 0)
     (effects (font (size 1.27 1.27)) (justify left bottom))
   )
@@
     (effects (font (size 1.2446 1.2446)) (justify right bottom))
   )
-  (label "I2C2_SCL" (at 43.18 49.53 180) (fields_autoplaced)
+  (label "I2C2_SCL" (at 48.26 40.64 180) (fields_autoplaced)
     (effects (font (size 1.2446 1.2446)) (justify right bottom))
   )
@@
     (effects (font (size 1.2446 1.2446)) (justify right bottom))
   )
-  (label "I2C2_SDA" (at 43.18 52.07 180) (fields_autoplaced)
+  (label "I2C2_SDA" (at 44.45 43.18 180) (fields_autoplaced)
     (effects (font (size 1.2446 1.2446)) (justify right bottom))
   )
@@
         (path "/72d5dd28-f3f0-4ab5-9534-b1d1ff89f7d5"
           (reference "#GND021") (unit 1)
+        )
+      )
+    )
+  )
+  (symbol (lib_id "Adafruit BMP388-eagle-import:RESISTOR_0603_NOOUT") (at 35.56 49.53 180) (unit 1)
+    (in_bom yes) (on_board yes) (dnp no)
+    (property "Reference" "R12" (at 35.56 46.99 0)
+      (effects (font (size 1.27 1.27)))
+    )
+    (property "Value" "4.7K" (at 35.56 49.53 0)
+      (effects (font (size 1.016 1.016) bold))
+    )
+    (property "Footprint" "Adafruit BMP388:0603-NO" (at 35.56 49.53 0)
+      (effects (font (size 1.27 1.27)) hide)
+    )
+    (property "Datasheet" "" (at 35.56 49.53 0)
+      (effects (font (size 1.27 1.27)) hide)
+    )
+    (pin "1")
+    (pin "2")
+    (instances
+      (project "air_station_1v5"
+        (path "/72d5dd28-f3f0-4ab5-9534-b1d1ff89f7d5"
+          (reference "R12") (unit 1)
         )
       )
@@
         (path "/72d5dd28-f3f0-4ab5-9534-b1d1ff89f7d5"
           (reference "C5") (unit 1)
+        )
+      )
+    )
+  )
+  (symbol (lib_id "Adafruit BMP388-eagle-import:3.3V") (at 25.4 44.45 0) (unit 1)
+    (in_bom yes) (on_board yes) (dnp no)
+    (property "Reference" "#U$04" (at 25.4 44.45 0)
+      (effects (font (size 1.27 1.27)) hide)
+    )
+    (property "Value" "3.3V" (at 23.876 43.434 0)
+      (effects (font (size 1.27 1.0795)) (justify left bottom))
+    )
+    (property "Footprint" "" (at 25.4 44.45 0)
+      (effects (font (size 1.27 1.27)) hide)
+    )
+    (property "Datasheet" "" (at 25.4 44.45 0)
+      (effects (font (size 1.27 1.27)) hide)
+    )
+    (pin "1")
+    (instances
+      (project "air_station_1v5"
+        (path "/72d5dd28-f3f0-4ab5-9534-b1d1ff89f7d5"
+          (reference "#U$04") (unit 1)
         )
       )
@@
         )
       )
+    )
+  )
+  (symbol (lib_id "Adafruit BMP388-eagle-import:RESISTOR_0603_NOOUT") (at 35.56 52.07 180) (unit 1)
+    (in_bom yes) (on_board yes) (dnp no)
+    (property "Reference" "R11" (at 35.56 54.61 0)
+      (effects (font (size 1.27 1.27)))
+    )
+    (property "Value" "4.7K" (at 35.56 52.07 0)
+      (effects (font (size 1.016 1.016) bold))
+    )
+    (property "Footprint" "Adafruit BMP388:0603-NO" (at 35.56 52.07 0)
+      (effects (font (size 1.27 1.27)) hide)
+    )
+    (property "Datasheet" "" (at 35.56 52.07 0)
+      (effects (font (size 1.27 1.27)) hide)
+    )
+    (pin "1")
+    (pin "2")
+    (instances
+      (project "air_station_1v5"
+        (path "/72d5dd28-f3f0-4ab5-9534-b1d1ff89f7d5"
+          (reference "R11") (unit 1)
+        )
+      )
